File: Cradle_Rocker_Board_RV01/Cradle_Rocker_Board_RV01.kicad_sch (KiCad schematic)
At the start: 13 parts, among them J1 Screw_Terminal_01x02, J2 Screw_Terminal_01x02, J3 Conn_01x04_Pin, Q1 NMOS, Q2 NMOS, Q3 NMOS

Commit message: This is actually just a coil test board.
Submitted RV01 to PCBWay for Fabrication and Assembly on 20240902
Parts:
- removed R1: 1R, Master_Resistors:R0603, symbol Device:R_Shunt_US
- added J4: Screw_Terminal_01x02, Master_Connectors:1984617_PHOENIX, symbol Connector:Screw_Terminal_01x02
- added R1: 3m, Master_Resistors:WSHP28183L000FEA_Vishay_Dale, symbol Device:R_US
- H1, H2, H3, H4: footprint (none) -> MountingHole:MountingHole_3.2mm_M3_DIN965_Pad
- J1, J2: footprint (none) -> Master_Connectors:1984617_PHOENIX; Manufacturer (none) -> Phoenix Contact; ManufacturerPN (none) -> 1984617
- J3: footprint (none) -> Master_Connectors:47053-1000_MOL
- Q1: footprint (none) -> Master_MOSFET:BSC014N04LSIATMA1; Manufacturer (none) -> Infineon Technologies; ManufacturerPN (none) -> BSC010N04LSIATMA1
- Q2, Q3: footprint (none) -> Master_MOSFET:DIO_RB558WMF_ROM-L; Manufacturer (none) -> Rohm Semiconductor; ManufacturerPN (none) -> RE1C002UNTCL
- R2, R3: Manufacturer (none) -> Panasonic Electronic Components; ManufacturerPN (none) -> ERJ-3EKF1001V
Connections:
- net GND: now also J4.2 (Pin_2)
- net coil+: now reaches J2.1 (Pin_1)
- net coil+: now also R1.2
- net coil-: now reaches J2.2 (Pin_2), Q1.3 (D)
- net VCC renamed VUSB
- net VUSB: now also J4.1 (Pin_1); no longer J1.1 (Pin_1)
- new net VBUS: J1.1 (Pin_1), R1.1
- no-connect marks 4 -> 2
Other:
- note added: "Level Shifter"
- note added: "NMOS for H-Bridge Coil Driver"
- note added: "nRF5340 Devkit"
- moved on the sheet: J1, J2
